File: hardware/valley.sch (KiCad schematic (older format))
At the start: 28 parts, among them IC1 ATMEGA1284P-A, P1 CONN_01X10, P2 USB_OTG, P3 CONN_02X03, P4 CONN_01X16, Q1 BSS138, Q2 BSS138, U1 CH340G, U2 AP111733, U3 TXS0108E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

Commit message: Moving LED to back of board.
Changed lines of the file:
@@
 Wire Wire Line
 	4050 5200 4200 5200
-Text GLabel 4200 6000 2    60   Output ~ 0
+Text GLabel 4200 5800 2    60   Output ~ 0
 LED_RED
 Text GLabel 4200 5900 2    60   Output ~ 0
 LED_GREEN
-Text GLabel 4200 5800 2    60   Output ~ 0
+Text GLabel 4200 6000 2    60   Output ~ 0
 LED_BLUE
 Text GLabel 5950 6100 0    60   Input ~ 0

Commit message: Updating schematic to link SDA/MOSI and SCL/SCK.
Parts:
- removed Q1: BSS138, cbrues/kicad-lib2/footprints/sm-ics.pretty:SM-SOT23, symbol BSS138
Connections:
- net labels removed: SCL, SDA
- wire segments 131 -> 122

Commit message: Removing some unnecessary pullup resistors.
Parts:
- removed R5, R6: 10k, Resistors_SMD:R_0805_HandSoldering, symbol R_Small
Connections:
- wire segments 122 -> 119
Changed lines of the file:
@@
 A0
-$Comp
-L R_Small R6
-U 1 1 58EB2116
-P 9950 6150
-F 0 "R6" H 10009 6196 50  0000 L CNN
-F 1 "10k" H 10009 6105 50  0000 L CNN
-F 2 "Resistors_SMD:R_0805_HandSoldering" H 9950 6150 50  0001 C CNN
-F 3 "" H 9950 6150 50  0000 C CNN
-	1    9950 6150
-	-1   0    0    1
-$EndComp
-$Comp
-L +3.3V #PWR023
-U 1 1 58EB2251
-P 9950 6400
-F 0 "#PWR023" H 9950 6250 50  0001 C CNN
-F 1 "+3.3V" H 9965 6573 50  0000 C CNN
-F 2 "" H 9950 6400 50  0000 C CNN
-F 3 "" H 9950 6400 50  0000 C CNN
-	1    9950 6400
-	0    1    1    0
-$EndComp
 $Comp
 L +3.3V #PWR024
@@
 	1    6200 6100
 	0    1    1    0
-$EndComp
-$Comp
-L GND #PWR026
-U 1 1 58EB4388
-P 9300 4300
-F 0 "#PWR026" H 9300 4050 50  0001 C CNN
-F 1 "GND" V 9305 4172 50  0000 R CNN
-F 2 "" H 9300 4300 50  0000 C CNN
-F 3 "" H 9300 4300 50  0000 C CNN
-	1    9300 4300
-	0    1    1    0
-$EndComp
-$Comp
-L R_Small R5
-U 1 1 58EB43FB
-P 9400 4400
-F 0 "R5" H 9459 4446 50  0000 L CNN
-F 1 "10k" H 9459 4355 50  0000 L CNN
-F 2 "Resistors_SMD:R_0805_HandSoldering" H 9400 4400 50  0001 C CNN
-F 3 "" H 9400 4400 50  0000 C CNN
-	1    9400 4400
-	1    0    0    -1
 $EndComp
 Text GLabel 9000 4500 0    60   Input ~ 0
@@
 	9000 4500 9550 4500
 Wire Wire Line
-	9300 4300 9400 4300
-Connection ~ 9400 4500
-Wire Wire Line
 	4050 4100 4200 4100
 Wire Wire Line
@@
 	8300 5350 8400 5350
 Wire Wire Line
-	8300 5750 8400 5750
-Wire Wire Line
 	9550 4950 10500 4950
 Wire Wire Line
@@
 Wire Wire Line
 	10400 4750 10500 4750
-Wire Wire Line
-	9550 5750 10500 5750
-Wire Wire Line
-	9950 6050 9950 5750
-Connection ~ 9950 5750
-Wire Wire Line
-	9950 6250 9950 6400
 Wire Wire Line
 	9550 5350 10500 5350
@@
 Wire Wire Line
 	10450 6250 10500 6250
+Wire Wire Line
+	9550 5750 10500 5750
+Wire Wire Line
+	8400 5750 8300 5750
 $EndSCHEMATC

Commit message: Updating schematics for wider trace width; 15mil is enough.
Changed lines of the file:
@@
 A0
 $Comp
-L +3.3V #PWR024
+L +3.3V #PWR023
 U 1 1 58EB28CE
 P 9550 5650
-F 0 "#PWR024" H 9550 5500 50  0001 C CNN
+F 0 "#PWR023" H 9550 5500 50  0001 C CNN
 F 1 "+3.3V" V 9550 5750 50  0000 L CNN
 F 2 "" H 9550 5650 50  0000 C CNN
@@
 $EndComp
 $Comp
-L +5V #PWR025
+L +5V #PWR024
 U 1 1 58EB29D6
 P 8300 5650
-F 0 "#PWR025" H 8300 5500 50  0001 C CNN
+F 0 "#PWR024" H 8300 5500 50  0001 C CNN
 F 1 "+5V" V 8315 5778 50  0000 L CNN
 F 2 "" H 8300 5650 50  0000 C CNN
@@
 L CONN_01X10 P1
 U 1 1 58EB6320
-P 4350 2950
-F 0 "P1" H 4428 2991 50  0000 L CNN
-F 1 "CONN_01X10" H 4428 2900 50  0000 L CNN
-F 2 "Pin_Headers:Pin_Header_Straight_1x10_Pitch2.54mm" H 4350 2950 50  0001 C CNN
-F 3 "" H 4350 2950 50  0000 C CNN
-	1    4350 2950
+P 4800 3150
+F 0 "P1" H 4878 3191 50  0000 L CNN
+F 1 "CONN_01X10" H 4878 3100 50  0000 L CNN
+F 2 "Pin_Headers:Pin_Header_Straight_1x10_Pitch2.54mm" H 4800 3150 50  0001 C CNN
+F 3 "" H 4800 3150 50  0000 C CNN
+	1    4800 3150
 	1    0    0    -1
 $EndComp
 $Comp
-L +5V #PWR027
+L +5V #PWR025
 U 1 1 58EB657C
-P 4050 2500
-F 0 "#PWR027" H 4050 2350 50  0001 C CNN
-F 1 "+5V" H 4065 2673 50  0000 C CNN
-F 2 "" H 4050 2500 50  0000 C CNN
-F 3 "" H 4050 2500 50  0000 C CNN
-	1    4050 2500
-	1    0    0    -1
-$EndComp
-$Comp
-L GND #PWR028
+P 4950 3500
+F 0 "#PWR025" H 4950 3350 50  0001 C CNN
+F 1 "+5V" H 4965 3673 50  0000 C CNN
+F 2 "" H 4950 3500 50  0000 C CNN
+F 3 "" H 4950 3500 50  0000 C CNN
+	1    4950 3500
+	0    1    1    0
+$EndComp
+$Comp
+L GND #PWR026
 U 1 1 58EB65DB
-P 4050 2600
-F 0 "#PWR028" H 4050 2350 50  0001 C CNN
-F 1 "GND" V 4055 2472 50  0000 R CNN
-F 2 "" H 4050 2600 50  0000 C CNN
-F 3 "" H 4050 2600 50  0000 C CNN
-	1    4050 2600
-	0    1    1    0
+P 4950 3600
+F 0 "#PWR026" H 4950 3350 50  0001 C CNN
+F 1 "GND" V 4955 3472 50  0000 R CNN
+F 2 "" H 4950 3600 50  0000 C CNN
+F 3 "" H 4950 3600 50  0000 C CNN
+	1    4950 3600
+	0    -1   -1   0
 $EndComp
 Wire Wire Line
@@
 	4050 6000 4200 6000
 Wire Wire Line
-	4050 2500 4150 2500
-Wire Wire Line
-	4150 2600 4050 2600
-Wire Wire Line
-	4050 2700 4150 2700
-Wire Wire Line
-	4150 2800 4050 2800
-Wire Wire Line
-	4050 2900 4150 2900
-Wire Wire Line
-	4050 3000 4150 3000
-Wire Wire Line
-	4150 3100 4050 3100
-Wire Wire Line
-	4050 3200 4150 3200
-Wire Wire Line
-	4150 3300 4050 3300
-Wire Wire Line
-	4050 3400 4150 3400
-Wire Wire Line
 	8400 5250 8300 5250
 Wire Wire Line
@@
 Wire Wire Line
 	8400 5750 8300 5750
+Wire Wire Line
+	4600 3500 4950 3500
+Wire Wire Line
+	4950 3600 4600 3600
+Wire Wire Line
+	4050 3400 4600 3400
+Wire Wire Line
+	4600 3300 4050 3300
+Wire Wire Line
+	4050 3200 4600 3200
+Wire Wire Line
+	4600 3100 4050 3100
+Wire Wire Line
+	4050 3000 4600 3000
+Wire Wire Line
+	4600 2900 4050 2900
+Wire Wire Line
+	4050 2800 4600 2800
+Wire Wire Line
+	4050 2700 4600 2700
 $EndSCHEMATC

Commit message: Updating schematic for v 1.1.
Parts:
- added C? (x2): 0.1u, symbol C
- added C?: 47u, cbrues/kicad-lib2/footprints/capacitors.pretty:SMD_PANASONIC_D, symbol CP
Connections:
- wire segments 119 -> 126
Changed lines of the file:
@@
 A0
-$Comp
-L +3.3V #PWR023
-U 1 1 58EB28CE
-P 9550 5650
-F 0 "#PWR023" H 9550 5500 50  0001 C CNN
-F 1 "+3.3V" V 9550 5750 50  0000 L CNN
-F 2 "" H 9550 5650 50  0000 C CNN
-F 3 "" H 9550 5650 50  0000 C CNN
-	1    9550 5650
-	0    1    1    0
-$EndComp
 $Comp
 L +5V #PWR024
 U 1 1 58EB29D6
-P 8300 5650
-F 0 "#PWR024" H 8300 5500 50  0001 C CNN
-F 1 "+5V" V 8315 5778 50  0000 L CNN
-F 2 "" H 8300 5650 50  0000 C CNN
-F 3 "" H 8300 5650 50  0000 C CNN
-	1    8300 5650
+P 7500 5650
+F 0 "#PWR024" H 7500 5500 50  0001 C CNN
+F 1 "+5V" V 7515 5778 50  0000 L CNN
+F 2 "" H 7500 5650 50  0000 C CNN
+F 3 "" H 7500 5650 50  0000 C CNN
+	1    7500 5650
 	0    -1   -1   0
 $EndComp
@@
 	8300 4850 8400 4850
 Wire Wire Line
-	8300 5650 8400 5650
+	7500 5650 8400 5650
 Wire Wire Line
 	6300 5700 6450 5700
@@
 Wire Wire Line
 	4050 2700 4600 2700
+$Comp
+L C C?
+U 1 1 58FCEB3F
+P 7600 5800
+F 0 "C?" H 7715 5846 50  0000 L CNN
+F 1 "0.1u" H 7715 5755 50  0000 L CNN
+F 2 "" H 7638 5650 50  0000 C CNN
+F 3 "" H 7600 5800 50  0000 C CNN
+	1    7600 5800
+	1    0    0    -1
+$EndComp
+$Comp
+L C C?
+U 1 1 58FCEC5F
+P 9650 6000
+F 0 "C?" H 9765 6046 50  0000 L CNN
+F 1 "0.1u" H 9765 5955 50  0000 L CNN
+F 2 "" H 9688 5850 50  0000 C CNN
+F 3 "" H 9650 6000 50  0000 C CNN
+	1    9650 6000
+	1    0    0    -1
+$EndComp
+$Comp
+L +3.3V #PWR?
+U 1 1 58FCECD9
+P 9750 5850
+F 0 "#PWR?" H 9750 5700 50  0001 C CNN
+F 1 "+3.3V" V 9750 5950 50  0000 L CNN
+F 2 "" H 9750 5850 50  0000 C CNN
+F 3 "" H 9750 5850 50  0000 C CNN
+	1    9750 5850
+	0    1    1    0
+$EndComp
+$Comp
+L GND #PWR?
+U 1 1 58FCEE19
+P 9650 6200
+F 0 "#PWR?" H 9650 5950 50  0001 C CNN
+F 1 "GND" V 9655 6072 50  0000 R CNN
+F 2 "" H 9650 6200 50  0000 C CNN
+F 3 "" H 9650 6200 50  0000 C CNN
+	1    9650 6200
+	1    0    0    -1
+$EndComp
+$Comp
+L GND #PWR?
+U 1 1 58FCEEC6
+P 7600 6000
+F 0 "#PWR?" H 7600 5750 50  0001 C CNN
+F 1 "GND" V 7605 5872 50  0000 R CNN
+F 2 "" H 7600 6000 50  0000 C CNN
+F 3 "" H 7600 6000 50  0000 C CNN
+	1    7600 6000
+	1    0    0    -1
+$EndComp
+Connection ~ 7600 5650
+Wire Wire Line
+	7600 6000 7600 5950
+Wire Wire Line
+	9650 5850 9650 5650
+Wire Wire Line
+	9650 5650 9550 5650
+Wire Wire Line
+	9650 6150 9650 6200
+Wire Wire Line
+	9750 5850 9650 5850
+$Comp
+L CP C?
+U 1 1 58FCF5C8
+P 9450 2950
+F 0 "C?" V 9705 2950 50  0000 C CNN
+F 1 "47u" V 9614 2950 50  0000 C CNN
+F 2 "cbrues/kicad-lib2/footprints/capacitors.pretty:SMD_PANASONIC_D" H 9488 2800 50  0001 C CNN
+F 3 "" H 9450 2950 50  0000 C CNN
+	1    9450 2950
+	1    0    0    -1
+$EndComp
+Wire Wire Line
+	9450 2700 9450 2800
+Wire Wire Line
+	9450 3100 8950 3100
+Connection ~ 8950 3100
 $EndSCHEMATC

Commit message: Adding latest schematic.
Parts:
- C11, C13: renamed from C?; footprint (none) -> Capacitors_SMD:C_0805_HandSoldering
- Y1: footprint tmk/keyboard_parts.pretty:HC-49_SMT -> monostable/CommonPartsLibrary.pretty:XTAL_HC-49US-16.000MHZ
- gave numbers to parts that had none: 1
Changed lines of the file:
@@
 F 0 "Y1" V 1604 3431 50  0000 L CNN
 F 1 "12M" V 1695 3431 50  0000 L CNN
-F 2 "tmk/keyboard_parts.pretty:HC-49_SMT" H 1650 3300 50  0001 C CNN
+F 2 "monostable/CommonPartsLibrary.pretty:XTAL_HC-49US-16.000MHZ" H 1650 3300 50  0001 C CNN
 F 3 "" H 1650 3300 50  0000 C CNN
 	1    1650 3300
@@
 A0
 $Comp
-L +5V #PWR024
+L +5V #PWR023
 U 1 1 58EB29D6
 P 7500 5650
-F 0 "#PWR024" H 7500 5500 50  0001 C CNN
+F 0 "#PWR023" H 7500 5500 50  0001 C CNN
 F 1 "+5V" V 7515 5778 50  0000 L CNN
 F 2 "" H 7500 5650 50  0000 C CNN
@@
 $EndComp
 $Comp
-L +5V #PWR025
+L +5V #PWR024
 U 1 1 58EB657C
 P 4950 3500
-F 0 "#PWR025" H 4950 3350 50  0001 C CNN
+F 0 "#PWR024" H 4950 3350 50  0001 C CNN
 F 1 "+5V" H 4965 3673 50  0000 C CNN
 F 2 "" H 4950 3500 50  0000 C CNN
@@
 $EndComp
 $Comp
-L GND #PWR026
+L GND #PWR025
 U 1 1 58EB65DB
 P 4950 3600
-F 0 "#PWR026" H 4950 3350 50  0001 C CNN
+F 0 "#PWR025" H 4950 3350 50  0001 C CNN
 F 1 "GND" V 4955 3472 50  0000 R CNN
 F 2 "" H 4950 3600 50  0000 C CNN
@@
 	4050 2700 4600 2700
 $Comp
-L C C?
+L C C11
 U 1 1 58FCEB3F
 P 7600 5800
-F 0 "C?" H 7715 5846 50  0000 L CNN
+F 0 "C11" H 7715 5846 50  0000 L CNN
 F 1 "0.1u" H 7715 5755 50  0000 L CNN
-F 2 "" H 7638 5650 50  0000 C CNN
+F 2 "Capacitors_SMD:C_0805_HandSoldering" H 7638 5650 50  0001 C CNN
 F 3 "" H 7600 5800 50  0000 C CNN
 	1    7600 5800
@@
 $EndComp
 $Comp
-L C C?
+L C C13
 U 1 1 58FCEC5F
 P 9650 6000
-F 0 "C?" H 9765 6046 50  0000 L CNN
+F 0 "C13" H 9765 6046 50  0000 L CNN
 F 1 "0.1u" H 9765 5955 50  0000 L CNN
-F 2 "" H 9688 5850 50  0000 C CNN
+F 2 "Capacitors_SMD:C_0805_HandSoldering" H 9688 5850 50  0001 C CNN
 F 3 "" H 9650 6000 50  0000 C CNN
 	1    9650 6000
@@
 $EndComp
 $Comp
-L +3.3V #PWR?
+L +3.3V #PWR026
 U 1 1 58FCECD9
 P 9750 5850
-F 0 "#PWR?" H 9750 5700 50  0001 C CNN
+F 0 "#PWR026" H 9750 5700 50  0001 C CNN
 F 1 "+3.3V" V 9750 5950 50  0000 L CNN
 F 2 "" H 9750 5850 50  0000 C CNN
@@
 $EndComp
 $Comp
-L GND #PWR?
+L GND #PWR027
 U 1 1 58FCEE19
 P 9650 6200
-F 0 "#PWR?" H 9650 5950 50  0001 C CNN
+F 0 "#PWR027" H 9650 5950 50  0001 C CNN
 F 1 "GND" V 9655 6072 50  0000 R CNN
 F 2 "" H 9650 6200 50  0000 C CNN
@@
 $EndComp
 $Comp
-L GND #PWR?
+L GND #PWR028
 U 1 1 58FCEEC6
 P 7600 6000
-F 0 "#PWR?" H 7600 5750 50  0001 C CNN
+F 0 "#PWR028" H 7600 5750 50  0001 C CNN
 F 1 "GND" V 7605 5872 50  0000 R CNN
 F 2 "" H 7600 6000 50  0000 C CNN
@@
 	9750 5850 9650 5850
 $Comp
-L CP C?
+L CP C12
 U 1 1 58FCF5C8
 P 9450 2950
-F 0 "C?" V 9705 2950 50  0000 C CNN
+F 0 "C12" V 9705 2950 50  0000 C CNN
 F 1 "47u" V 9614 2950 50  0000 C CNN
 F 2 "cbrues/kicad-lib2/footprints/capacitors.pretty:SMD_PANASONIC_D" H 9488 2800 50  0001 C CNN

Commit message: Updating to latest kicad version before next iteration.
Parts:
- P2: symbol USB_OTG -> USB_OTG-RESCUE-valley
- Q2: symbol BSS138 -> BSS138-RESCUE-valley
Changed lines of the file:
@@
-EESchema Schematic File Version 2
+EESchema Schematic File Version 3
+LIBS:valley-rescue
 LIBS:power
 LIBS:device
@@
 CLKO
 $Comp
-L USB_OTG P2
+L USB_OTG-RESCUE-valley P2
 U 1 1 58EAD0A2
 P 5050 2650
@@
 $EndComp
 $Comp
-L BSS138 Q2
+L BSS138-RESCUE-valley Q2
 U 1 1 58EB0E1D
 P 10000 4600

Commit message: ESP12E version laid out.
Parts:
- removed C10, C11, C13, C9: 0.1u, Capacitors_SMD:C_0805_HandSoldering, symbol C
- removed C7: 47u, cbrues/kicad-lib2/footprints/capacitors.pretty:SMD_PANASONIC_D, symbol CP
- removed IC1: ATMEGA1284P-A, OLIMEX/KiCAD/KiCAD_Footprints/OLIMEX_IC-FP.pretty:TQFP44, symbol ATMEGA1284P-A
- removed P1: CONN_01X10, Pin_Headers:Pin_Header_Straight_1x10_Pitch2.54mm, symbol CONN_01X10
- removed P3: CONN_02X03, Pin_Headers:Pin_Header_Straight_2x03_Pitch2.54mm_SMD, symbol CONN_02X03
- removed R1: 10k, Resistors_SMD:R_0805_HandSoldering, symbol R_Small
- removed R2, R3: 1.5k, Resistors_SMD:R_0805_HandSoldering, symbol R_Small
- removed R4: 1k, Resistors_SMD:R_0805_HandSoldering, symbol R_Small
- removed U1: CH340G, Housings_SOIC:SOIC-16_3.9x9.9mm_Pitch1.27mm, symbol CH340G
- removed U3: TXS0108E, Housings_SSOP:TSSOP-20_4.4x6.5mm_Pitch0.65mm, symbol TXS0108E
- added ??1: PCA9557, adamgreig/agg-kicad/agg.pretty:SOIC-16, symbol PCA9557
- added IC1: TLC5971_SOP, brunoeagle/kicad-open-modules:TSSOP-20, symbol TLC5971_SOP
- added Q1, Q3: PDTD113ZT,215, celeritous/KiCad.pretty:SOT23-3, symbol 2N3055
- added R1: R, coddingtonbear/coddingtonbear.pretty:0805_Milling, symbol R
- added R2, R3, R8, R9: 10k, coddingtonbear/coddingtonbear.pretty:0805_Milling, symbol R
- added R4: 5k, coddingtonbear/coddingtonbear.pretty:0805_Milling, symbol R
- added R5: 2k, coddingtonbear/coddingtonbear.pretty:0805_Milling, symbol R
- added R6: 100k, coddingtonbear/coddingtonbear.pretty:0805_Milling, symbol R
- added R7: 4.7k, coddingtonbear/coddingtonbear.pretty:0805_Milling, symbol R
- added U1: CH341A, KiCad/SMD_Packages.pretty:SOIC-28, symbol CH341A
- added U3: ESP-12E, coddingtonbear/coddingtonbear.pretty:ESP-12E, symbol ESP-12E
- C1, C2, C3, C4, C5, C6, C8: footprint Capacitors_SMD:C_0805_HandSoldering -> coddingtonbear/coddingtonbear.pretty:0805_Milling
- C12: value 47u -> 1000u; footprint cbrues/kicad-lib2/footprints/capacitors.pretty:SMD_PANASONIC_D -> ohdsp/KiCad-Libs/MyKiCadLibs-Footprints.pretty:CAP-SMD-SIZE-F
- P2: footprint valley:MICRO-B_USB-INVERTED -> coddingtonbear/coddingtonbear.pretty:UJ2-MIBH-4-SMT
Connections:
- net labels added: DTR, GPIO0, REST, RTS, SCL, SDA, UD+, UD-
- net labels removed: CLKO, ENABLE_LC, RESET
- wire segments 126 -> 108
Other:
- note added: "DTR/RST Reset Handler; adapted from\nnodemcu/nodemcu-devkit/master/Documents/NODEMCU_DEVKIT_SCH.png"
- moved on the sheet: P2
