File: hardware/valley.sch (KiCad schematic (older format))
At the start: 29 parts, among them IC1 TLC5971_SOP, P2 USB_OTG, P4 CONN_01X16, Q1 PDTD113ZT,215, Q2 BSS138, Q3 PDTD113ZT,215, U1 CH341A, U2 AP111733, U3 ESP-12E, Y1 12M

Commit message: Updating to use ESP32 as main processor -- no need of the separate LED driver or I2C IO expander.
Parts:
- removed ??1: PCA9557, adamgreig/agg-kicad/agg.pretty:SOIC-16, symbol PCA9557
- removed C4, C5, C6, C8: 0.1u, coddingtonbear/coddingtonbear.pretty:0805_Milling, symbol C
- removed IC1: TLC5971_SOP, brunoeagle/kicad-open-modules:TSSOP-20, symbol TLC5971_SOP
- removed Q1, Q3: PDTD113ZT,215, celeritous/KiCad.pretty:SOT23-3, symbol 2N3055
- removed R2, R8, R9: 10k, coddingtonbear/coddingtonbear.pretty:0805_Milling, symbol R
- removed R6: 100k, coddingtonbear/coddingtonbear.pretty:0805_Milling, symbol R
- removed U1: CH341A, KiCad/SMD_Packages.pretty:SOIC-28, symbol CH341A
- removed U3: ESP-12E, coddingtonbear/coddingtonbear.pretty:ESP-12E, symbol ESP-12E
- added U1: CH340G, adamgreig/agg-kicad/agg.pretty:SOIC-16, symbol CH340G
- added U3: ESP32-WROOM, adamjvr/ESP32-kiCAD-Footprints/ESP32-Footprints/ESP32-footprints-Lib.pretty:ESP32-WROOM, symbol ESP32-WROOM
- D1: footprint valley:SLV6A-FKB -> coddingtonbear/coddingtonbear.pretty:SLV6A-FKB-MILLING
- R1: value R -> 10k
- R4: value 5k -> 10k
- R5: value 2k -> 10k
- R7: value 4.7k -> 10k
- Y1: footprint monostable/CommonPartsLibrary.pretty:XTAL_HC-49US-16.000MHZ -> KiCad/Crystals.pretty:Crystal_SMD_HC49-SD_HandSoldering
Connections:
- net labels removed: GPIO0, REST, SCL, SDA
- wire segments 108 -> 59
Other:
- note removed: "DTR/RST Reset Handler; adapted from\nnodemcu/nodemcu-devkit/master/Documents/NODEMCU_DEVKIT_SCH.png"
- moved on the sheet: P2

Commit message: Swapping CH340G to CH341A
Parts:
- removed U1: CH340G, adamgreig/agg-kicad/agg.pretty:SOIC-16, symbol CH340G
- added U1: CH341A, KiCad/Housings_SOIC.pretty:SOIC-28W_7.5x17.9mm_Pitch1.27mm, symbol CH341A
- Q2: footprint cbrues/kicad-lib2/footprints/sm-ics.pretty:SM-SOT23 -> KiCad/TO_SOT_Packages_SMD.pretty:SOT-23_Handsoldering
Connections:
- net labels added: BACKLIGHT_3V3, USB_CONNECTED
- wire segments 59 -> 63
Changed lines of the file:
@@
 L Crystal Y1
 U 1 1 58EAC422
-P 1700 3950
-F 0 "Y1" V 1654 4081 50  0000 L CNN
-F 1 "12M" V 1745 4081 50  0000 L CNN
-F 2 "KiCad/Crystals.pretty:Crystal_SMD_HC49-SD_HandSoldering" H 1700 3950 50  0001 C CNN
-F 3 "" H 1700 3950 50  0000 C CNN
-	1    1700 3950
+P 1600 3250
+F 0 "Y1" V 1554 3381 50  0000 L CNN
+F 1 "12M" V 1645 3381 50  0000 L CNN
+F 2 "KiCad/Crystals.pretty:Crystal_SMD_HC49-SD_HandSoldering" H 1600 3250 50  0001 C CNN
+F 3 "" H 1600 3250 50  0000 C CNN
+	1    1600 3250
 	0    1    1    0
 $EndComp
@@
 F 0 "Q2" H 10191 4646 50  0000 L CNN
 F 1 "BSS138" H 10191 4555 50  0000 L CNN
-F 2 "cbrues/kicad-lib2/footprints/sm-ics.pretty:SM-SOT23" H 10200 4525 50  0001 L CIN
+F 2 "KiCad/TO_SOT_Packages_SMD.pretty:SOT-23_Handsoldering" H 10200 4525 50  0001 L CIN
 F 3 "" H 10000 4600 50  0000 L CNN
 	1    10000 4600
@@
 L C C1
 U 1 1 59D96260
-P 1550 3800
-F 0 "C1" V 1298 3800 50  0000 C CNN
-F 1 "22p" V 1389 3800 50  0000 C CNN
-F 2 "coddingtonbear/coddingtonbear.pretty:0805_Milling" H 1588 3650 50  0001 C CNN
-F 3 "" H 1550 3800 50  0000 C CNN
-	1    1550 3800
+P 1450 3100
+F 0 "C1" V 1198 3100 50  0000 C CNN
+F 1 "22p" V 1289 3100 50  0000 C CNN
+F 2 "coddingtonbear/coddingtonbear.pretty:0805_Milling" H 1488 2950 50  0001 C CNN
+F 3 "" H 1450 3100 50  0000 C CNN
+	1    1450 3100
 	0    -1   -1   0
 $EndComp
@@
 L C C2
 U 1 1 59D962BF
-P 1550 4100
-F 0 "C2" V 1298 4100 50  0000 C CNN
-F 1 "22p" V 1389 4100 50  0000 C CNN
-F 2 "coddingtonbear/coddingtonbear.pretty:0805_Milling" H 1588 3950 50  0001 C CNN
-F 3 "" H 1550 4100 50  0000 C CNN
-	1    1550 4100
+P 1450 3400
+F 0 "C2" V 1198 3400 50  0000 C CNN
+F 1 "22p" V 1289 3400 50  0000 C CNN
+F 2 "coddingtonbear/coddingtonbear.pretty:0805_Milling" H 1488 3250 50  0001 C CNN
+F 3 "" H 1450 3400 50  0000 C CNN
+	1    1450 3400
 	0    -1   -1   0
 $EndComp
@@
 L GND #PWR01
 U 1 1 59D9659A
-P 1350 3950
-F 0 "#PWR01" H 1350 3700 50  0001 C CNN
-F 1 "GND" H 1355 3777 50  0000 C CNN
-F 2 "" H 1350 3950 50  0000 C CNN
-F 3 "" H 1350 3950 50  0000 C CNN
-	1    1350 3950
-	0    1    1    0
-$EndComp
-Text GLabel 2100 3600 0    60   BiDi ~ 0
+P 1250 3250
+F 0 "#PWR01" H 1250 3000 50  0001 C CNN
+F 1 "GND" H 1255 3077 50  0000 C CNN
+F 2 "" H 1250 3250 50  0000 C CNN
+F 3 "" H 1250 3250 50  0000 C CNN
+	1    1250 3250
+	0    1    1    0
+$EndComp
+Text GLabel 2000 3450 0    60   BiDi ~ 0
 UD+
-Text GLabel 2100 3700 0    60   BiDi ~ 0
+Text GLabel 2000 3550 0    60   BiDi ~ 0
 UD-
 Text GLabel 2700 1450 2    60   BiDi ~ 0
@@
 	0    1    1    0
 $EndComp
-Text GLabel 3100 3800 2    60   Input ~ 0
+Text GLabel 3200 3850 2    60   Input ~ 0
 TXD
-Text GLabel 3100 3900 2    60   Output ~ 0
+Text GLabel 3200 3750 2    60   Output ~ 0
 RXD
 Text GLabel 7500 1950 2    60   Output ~ 0
@@
 	1    0    0    -1
 $EndComp
-Text GLabel 3100 4300 2    60   BiDi ~ 0
+Text GLabel 3200 4650 2    60   BiDi ~ 0
 DTR
-Text GLabel 3100 4100 2    60   BiDi ~ 0
+Text GLabel 3200 4750 2    60   BiDi ~ 0
 RTS
 Text GLabel 8050 3000 2    60   BiDi ~ 0
@@
 	0    1    1    0
 $EndComp
-$Comp
-L CH340G U1
-U 1 1 59F299D6
-P 2600 4200
-F 0 "U1" H 2600 5087 60  0000 C CNN
-F 1 "CH340G" H 2600 4981 60  0000 C CNN
-F 2 "adamgreig/agg-kicad/agg.pretty:SOIC-16" H 2550 5300 60  0001 C CNN
-F 3 "" H 2550 5300 60  0000 C CNN
-	1    2600 4200
-	1    0    0    -1
-$EndComp
-Wire Wire Line
-	2100 3900 1850 3900
-Wire Wire Line
-	1850 3900 1850 3800
-Wire Wire Line
-	1850 3800 1700 3800
-Wire Wire Line
-	2100 4000 1850 4000
-Wire Wire Line
-	1850 4000 1850 4100
-Wire Wire Line
-	1850 4100 1700 4100
-Wire Wire Line
-	1400 3800 1400 4100
-Wire Wire Line
-	1400 3950 1350 3950
-Connection ~ 1400 3950
+Wire Wire Line
+	2000 3200 1750 3200
+Wire Wire Line
+	1750 3200 1750 3100
+Wire Wire Line
+	1750 3100 1600 3100
+Wire Wire Line
+	2000 3300 1750 3300
+Wire Wire Line
+	1750 3300 1750 3400
+Wire Wire Line
+	1750 3400 1600 3400
+Wire Wire Line
+	1300 3100 1300 3400
+Wire Wire Line
+	1300 3250 1250 3250
+Connection ~ 1300 3250
 $Comp
 L C C3
 U 1 1 59F2A45F
-P 3200 3450
-F 0 "C3" V 2948 3450 50  0000 C CNN
-F 1 "0.1u" V 3039 3450 50  0000 C CNN
-F 2 "coddingtonbear/coddingtonbear.pretty:0805_Milling" H 3238 3300 50  0001 C CNN
-F 3 "" H 3200 3450 50  0000 C CNN
-	1    3200 3450
+P 3400 3050
+F 0 "C3" V 3148 3050 50  0000 C CNN
+F 1 "0.1u" V 3239 3050 50  0000 C CNN
+F 2 "coddingtonbear/coddingtonbear.pretty:0805_Milling" H 3438 2900 50  0001 C CNN
+F 3 "" H 3400 3050 50  0000 C CNN
+	1    3400 3050
 	-1   0    0    1
 $EndComp
@@
 L +3.3V #PWR04
 U 1 1 59F2A4D1
-P 3350 3600
-F 0 "#PWR04" H 3350 3450 50  0001 C CNN
-F 1 "+3.3V" H 3365 3773 50  0000 C CNN
-F 2 "" H 3350 3600 50  0000 C CNN
-F 3 "" H 3350 3600 50  0000 C CNN
-	1    3350 3600
+P 3550 3200
+F 0 "#PWR04" H 3550 3050 50  0001 C CNN
+F 1 "+3.3V" H 3565 3373 50  0000 C CNN
+F 2 "" H 3550 3200 50  0000 C CNN
+F 3 "" H 3550 3200 50  0000 C CNN
+	1    3550 3200
 	0    1    1    0
 $EndComp
@@
 L GND #PWR05
 U 1 1 59F2A527
-P 3350 3300
-F 0 "#PWR05" H 3350 3050 50  0001 C CNN
-F 1 "GND" H 3355 3127 50  0000 C CNN
-F 2 "" H 3350 3300 50  0000 C CNN
-F 3 "" H 3350 3300 50  0000 C CNN
-	1    3350 3300
+P 3550 2850
+F 0 "#PWR05" H 3550 2600 50  0001 C CNN
+F 1 "GND" H 3555 2677 50  0000 C CNN
+F 2 "" H 3550 2850 50  0000 C CNN
+F 3 "" H 3550 2850 50  0000 C CNN
+	1    3550 2850
 	0    -1   -1   0
 $EndComp
-$Comp
-L +3.3V #PWR09
-U 1 1 59F2A5AF
-P 2000 4300
-F 0 "#PWR09" H 2000 4150 50  0001 C CNN
-F 1 "+3.3V" H 2015 4473 50  0000 C CNN
-F 2 "" H 2000 4300 50  0000 C CNN
-F 3 "" H 2000 4300 50  0000 C CNN
-	1    2000 4300
-	0    -1   -1   0
-$EndComp
-Wire Wire Line
-	3100 3600 3350 3600
-Connection ~ 3200 3600
-Wire Wire Line
-	3350 3300 3200 3300
-Wire Wire Line
-	2000 4300 2100 4300
 $Comp
 L GND #PWR026
 U 1 1 59F2A8D5
-P 3100 4700
-F 0 "#PWR026" H 3100 4450 50  0001 C CNN
-F 1 "GND" H 3105 4527 50  0000 C CNN
-F 2 "" H 3100 4700 50  0000 C CNN
-F 3 "" H 3100 4700 50  0000 C CNN
-	1    3100 4700
+P 3200 3400
+F 0 "#PWR026" H 3200 3150 50  0001 C CNN
+F 1 "GND" H 3205 3227 50  0000 C CNN
+F 2 "" H 3200 3400 50  0000 C CNN
+F 3 "" H 3200 3400 50  0000 C CNN
+	1    3200 3400
 	1    0    0    -1
 $EndComp
@@
 Wire Wire Line
 	5750 6950 5800 6950
+Wire Wire Line
+	7500 2950 7500 3050
+$Comp
+L CH341A U1
+U 1 1 59F3DECD
+P 2600 3750
+F 0 "U1" H 2600 4587 60  0000 C CNN
+F 1 "CH341A" H 2600 4481 60  0000 C CNN
+F 2 "KiCad/Housings_SOIC.pretty:SOIC-28W_7.5x17.9mm_Pitch1.27mm" H 2550 4850 60  0001 C CNN
+F 3 "" H 2550 4850 60  0000 C CNN
+	1    2600 3750
+	1    0    0    -1
+$EndComp
+Wire Wire Line
+	3200 3200 3550 3200
+Connection ~ 3400 3200
+Wire Wire Line
+	3400 2900 3400 2850
+Wire Wire Line
+	3400 2850 3550 2850
+$Comp
+L GND #PWR07
+U 1 1 59F3E5A2
+P 1750 3800
+F 0 "#PWR07" H 1750 3550 50  0001 C CNN
+F 1 "GND" H 1755 3627 50  0000 C CNN
+F 2 "" H 1750 3800 50  0000 C CNN
+F 3 "" H 1750 3800 50  0000 C CNN
+	1    1750 3800
+	1    0    0    -1
+$EndComp
+Wire Wire Line
+	1750 3800 2000 3800
+Text GLabel 7500 2050 2    60   Input ~ 0
+USB_CONNECTED
+Text GLabel 2000 3650 0    60   Output ~ 0
+USB_CONNECTED
+Wire Wire Line
+	3200 3300 3400 3300
+Wire Wire Line
+	3400 3300 3400 3200
+Text Label 10100 4850 0    60   ~ 0
+BACKLIGHT_3V3
 $EndSCHEMATC

Commit message: Minor schematic updates.
Parts:
- removed Q2: BSS138, KiCad/TO_SOT_Packages_SMD.pretty:SOT-23_Handsoldering, symbol BSS138-RESCUE-valley
- R1, R4: value 10k -> 10
- R5: value 10k -> 150
Connections:
- net labels removed: BACKLIGHT, BACKLIGHT_3V3
- wire segments 63 -> 59
Changed lines of the file:
@@
 CS_TFT
-$Comp
-L BSS138-RESCUE-valley Q2
-U 1 1 58EB0E1D
-P 10000 4600
-F 0 "Q2" H 10191 4646 50  0000 L CNN
-F 1 "BSS138" H 10191 4555 50  0000 L CNN
-F 2 "KiCad/TO_SOT_Packages_SMD.pretty:SOT-23_Handsoldering" H 10200 4525 50  0001 L CIN
-F 3 "" H 10000 4600 50  0000 L CNN
-	1    10000 4600
-	1    0    0    -1
-$EndComp
 $Comp
 L +3.3V #PWR021
 U 1 1 58EB0EAB
-P 10100 4250
-F 0 "#PWR021" H 10100 4100 50  0001 C CNN
-F 1 "+3.3V" H 10115 4423 50  0000 C CNN
-F 2 "" H 10100 4250 50  0000 C CNN
-F 3 "" H 10100 4250 50  0000 C CNN
-	1    10100 4250
-	1    0    0    -1
-$EndComp
-Text GLabel 7500 2650 2    60   Output ~ 0
-BACKLIGHT
-Text GLabel 9750 4550 1    60   Input ~ 0
-BACKLIGHT
+P 10100 4850
+F 0 "#PWR021" H 10100 4700 50  0001 C CNN
+F 1 "+3.3V" H 10115 5023 50  0000 C CNN
+F 2 "" H 10100 4850 50  0000 C CNN
+F 3 "" H 10100 4850 50  0000 C CNN
+	1    10100 4850
+	0    -1   -1   0
+$EndComp
 Text GLabel 9550 5450 0    60   Input ~ 0
 A0
@@
 	9550 4950 10500 4950
 Wire Wire Line
-	10500 4850 10100 4850
-Wire Wire Line
-	10100 4850 10100 4800
-Wire Wire Line
-	9800 4650 9750 4650
-Wire Wire Line
-	9750 4650 9750 4550
-Wire Wire Line
-	10100 4250 10100 4400
+	10100 4850 10500 4850
 Wire Wire Line
 	10400 4750 10500 4750
@@
 P 5600 6550
 F 0 "R1" V 5393 6550 50  0000 C CNN
-F 1 "10k" V 5484 6550 50  0000 C CNN
+F 1 "10" V 5484 6550 50  0000 C CNN
 F 2 "coddingtonbear/coddingtonbear.pretty:0805_Milling" V 5530 6550 50  0001 C CNN
 F 3 "" H 5600 6550 50  0001 C CNN
@@
 P 5600 6750
 F 0 "R4" V 5393 6750 50  0000 C CNN
-F 1 "10k" V 5484 6750 50  0000 C CNN
+F 1 "10" V 5484 6750 50  0000 C CNN
 F 2 "coddingtonbear/coddingtonbear.pretty:0805_Milling" V 5530 6750 50  0001 C CNN
 F 3 "" H 5600 6750 50  0001 C CNN
@@
 P 5600 6950
 F 0 "R5" V 5393 6950 50  0000 C CNN
-F 1 "10k" V 5484 6950 50  0000 C CNN
+F 1 "150" V 5484 6950 50  0000 C CNN
 F 2 "coddingtonbear/coddingtonbear.pretty:0805_Milling" V 5530 6950 50  0001 C CNN
 F 3 "" H 5600 6950 50  0001 C CNN
@@
 Wire Wire Line
 	3400 3300 3400 3200
-Text Label 10100 4850 0    60   ~ 0
-BACKLIGHT_3V3
 $EndSCHEMATC
